Commit message: lidar plugin

File: husky_ur5/urdf/husky_ur5.urdf.xacro (robot description, xacro)
@@ -235,3 +235,8 @@
     <origin xyz="0 0 0" rpy="0 ${-pi/2} 0"/>
   </xacro:robotiq_85_gripper>
+  <!-- lidar -->
+  <xacro:include filename="$(find husky_ur5)/urdf/3d_lidar.urdf.xacro" />
+  <xacro:velodyne_lidar name="front_laser" topic="$(arg robot_namespace)/points" parent="base_link" max_range="75" update_rate="15">
+      <origin xyz="0.45 0.0 0.325" rpy="0 0 0"/>
+  </xacro:velodyne_lidar>
 </robot>

File: husky_ur5/urdf/husky_ur5_contact.urdf.xacro (robot description, xacro)
@@ -276,3 +276,8 @@
     <origin xyz="0 0 0" rpy="0 ${-pi/2} 0"/>
   </xacro:robotiq_85_gripper>
+  <!-- lidar -->
+  <xacro:include filename="$(find husky_ur5)/urdf/3d_lidar.urdf.xacro" />
+  <xacro:velodyne_lidar name="front_laser" topic="$(arg robot_namespace)/points" parent="base_link" max_range="75" update_rate="15">
+      <origin xyz="0.45 0.0 0.325" rpy="0 0 0"/>
+  </xacro:velodyne_lidar>
 </robot>
